File: shema.sch (EAGLE design)
At the start: 14 parts

Commit message: фиксы
Parts:
- removed U$7: TRAN_P, 1_TRANSISTOR (2):TRAN_P
- added VT1: TRAN_P, 1_TRANSISTOR (2):TRAN_P
- U$6: value RESISTOR0603 -> 0.015
Connections:
- net N$13 renamed 8.4V
- net N$3 renamed V_IN
- removed net N$2: U$12.S
- net GND: now also U$12.S
- net N$10: now also VT1.G; no longer U$7.G
- net N$4: now also VT1.S; no longer U$7.S
- net N$5: now also VT1.D; no longer U$7.D
Other:
- moved on the sheet: DD1, U$10, U$11, U$12, U$2, U$3, U$4, U$5, U$8, U$9

Commit message: добавила файлы
Parts:
- removed U$10: INDUCTOR, 1_NDUCTORS:INDUCTOR
- removed U$12: TRANSISTORN, 1_TRANSISTOR (2):TRANSISTORN
- removed U$14, U$2, U$3: RESISTOR0603, 1_RESISTOR:RESISTOR0603
- removed U$4, U$5: LED, 1_LED:LED
- removed U$8: B560C-13-F, 1_DIOD:B560C-13-F
- removed U$9: CAPACITOR, 1_RESISTOR:CAPACITOR
- added C0: 22uF, 1_RESISTOR:CAPACITOR
- added D1: B560C-13-F, 1_DIOD:B560C-13-F
- added D3, D4: LED, 1_LED:LED
- added L1: INDUCTOR, 1_NDUCTORS:INDUCTOR
- added M1: TRANSISTORN, 1_TRANSISTOR (2):TRANSISTORN
- added R1, R2, R3: RESISTOR0603, 1_RESISTOR:RESISTOR0603
- C1: value CAPACITOR -> 22uF
- renumbered U$1 to C1, U$11 to D2, U$6 to RCS, VT1 to M2
Connections:
- net 8.4V: now also C0.1, D1.C; no longer U$8.C, U$9.1
- net GND: now also C0.2, D4.C, M1.S; no longer U$12.S, U$5.C, U$9.2
- net N$1: now also D4.A, R2.P$1; no longer U$3.P$1, U$5.A
- net N$11: now also D3.C, R2.P$2; no longer U$3.P$2, U$4.C
- net N$12: now also D3.A, R1.P$1; no longer U$2.P$1, U$4.A
- net N$5: now also L1.1; no longer U$10.1
- net N$6: now also D1.A, L1.2, M1.D; no longer U$10.2, U$12.D, U$8.A
- net N$8: now also R3.P$2; no longer U$14.P$2
- net N$9: now also M1.G, R3.P$1; no longer U$12.G, U$14.P$1
- net V_IN: now also R1.P$2; no longer U$2.P$2

Commit message: файлы изменение
Connections:
- removed net CE: DD1.CE
- removed net VIN: DD1.VIN
- net V_IN: now also DD1.CE, DD1.VIN
Other:
- moved on the sheet: C0, D1, D2, D3, D4, M2, R1, R2, R3, RCS

Commit message: fix
Parts:
- R3: value RESISTOR0603 -> 1.8
- RCS: device 1_RESISTOR:RESISTOR0603 -> 1_RESISTOR:RESISTOR
Connections:
- net 8.4V: now also DD1.BAT
- net GND: no longer DD1.BAT
Other:
- moved on the sheet: C0, D1, D2, L1, M1, M2, R3, RCS

Commit message: файлы изменение
Parts:
- added C2, C3, C4, C5, C6, C7: 22uF, 1_RESISTOR:CAPACITOR
- RCS: device 1_RESISTOR:RESISTOR -> 1_RESISTOR:RESISTOR0603
Connections:
- new net N$15: C5.2, C6.1
- new net N$16: C0.2, C7.1
- new net N$2: C2.2, C3.1
- new net N$3: C1.2, C4.1
- new net N$7: C3.2, C4.2, R1.P$2
- net 8.4V: now also C5.1
- net GND: now also C6.2, C7.2; no longer C0.2, C1.2
- net V_IN: now also C2.1; no longer R1.P$2
Other:
- moved on the sheet: C0, C1, D1, D2, D3, D4, DD1, L1, M1, M2, R1, R2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

Commit message: файлы изменение
Parts:
- removed R1, R2: RESISTOR0603, 1_RESISTOR:RESISTOR0603
- removed R3: 1.8, 1_RESISTOR:RESISTOR0603
- added R4, R5: RESISTOR, 1_RESISTOR:RESISTOR
- added R6: 1.8, 1_RESISTOR:RESISTOR
- renumbered D3 to LED1, D4 to LED2, M1 to TV1, M2 to TV2
Connections:
- net N$1: now also R5.P$1; no longer R2.P$1
- net N$11: now also R5.P$2; no longer R2.P$2
- net N$12: now also R4.P$1; no longer R1.P$1
- net N$7: now also R4.P$2; no longer R1.P$2
- net N$8: now also R6.P$2; no longer R3.P$2
- net N$9: now also R6.P$1; no longer R3.P$1
Changed lines of the file:
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@@
 <part name="DD1" library="1_MICRO" deviceset="CN3302" device=""/>
 <part name="C1" library="1_RESISTOR" deviceset="CAPACITOR" device="" value="22uF"/>
-<part name="R1" library="1_RESISTOR" deviceset="RESISTOR" device="0603"/>
-<part name="R2" library="1_RESISTOR" deviceset="RESISTOR" device="0603"/>
 <part name="D1" library="1_DIOD" deviceset="B560C-13-F" device=""/>
 <part name="C0" library="1_RESISTOR" deviceset="CAPACITOR" device="" value="22uF"/>
 <part name="L1" library="1_NDUCTORS" deviceset="INDUCTOR" device=""/>
 <part name="D2" library="1_DIOD" deviceset="SS36C" device=""/>
-<part name="M1" library="1_TRANSISTOR (2)" deviceset="TRANSISTORN" device=""/>
-<part name="D3" library="1_LED" deviceset="LED" device=""/>
-<part name="D4" library="1_LED" deviceset="LED" device=""/>
-<part name="R3" library="1_RESISTOR" deviceset="RESISTOR" device="0603" value="1.8"/>
+<part name="TV1" library="1_TRANSISTOR (2)" deviceset="TRANSISTORN" device=""/>
+<part name="LED1" library="1_LED" deviceset="LED" device=""/>
+<part name="LED2" library="1_LED" deviceset="LED" device=""/>
 <part name="RCS" library="1_RESISTOR" deviceset="RESISTOR" device="0603" value="0.015"/>
-<part name="M2" library="1_TRANSISTOR (2)" deviceset="TRAN_P" device=""/>
+<part name="TV2" library="1_TRANSISTOR (2)" deviceset="TRAN_P" device=""/>
 <part name="C2" library="1_RESISTOR" deviceset="CAPACITOR" device="" value="22uF"/>
 <part name="C3" library="1_RESISTOR" deviceset="CAPACITOR" device="" value="22uF"/>
@@
 <part name="C6" library="1_RESISTOR" deviceset="CAPACITOR" device="" value="22uF"/>
 <part name="C7" library="1_RESISTOR" deviceset="CAPACITOR" device="" value="22uF"/>
+<part name="R4" library="1_RESISTOR" deviceset="RESISTOR" device=""/>
+<part name="R5" library="1_RESISTOR" deviceset="RESISTOR" device=""/>
+<part name="R6" library="1_RESISTOR" deviceset="RESISTOR" device="" value="1.8"/>
 </parts>
 <sheets>
@@
 <attribute name="VALUE" x="-39.116" y="30.861" size="1.778" layer="96"/>
 </instance>
-<instance part="R1" gate="G$1" x="-38.1" y="12.7" smashed="yes" rot="R90">
-<attribute name="VALUE" x="-35.306" y="9.906" size="1.27" layer="96" rot="R90"/>
-<attribute name="NAME" x="-40.132" y="9.652" size="1.27" layer="95" rot="R90"/>
-</instance>
-<instance part="R2" gate="G$1" x="-38.1" y="-12.7" smashed="yes" rot="R90">
-<attribute name="VALUE" x="-35.306" y="-15.494" size="1.27" layer="96" rot="R90"/>
-<attribute name="NAME" x="-40.132" y="-15.748" size="1.27" layer="95" rot="R90"/>
-</instance>
 <instance part="D1" gate="G$1" x="55.88" y="40.64" smashed="yes">
 <attribute name="NAME" x="53.34" y="43.18" size="1.778" layer="95"/>
@@
 <attribute name="VALUE" x="34.9758" y="30.4546" size="1.778" layer="96" rot="R90"/>
 </instance>
-<instance part="M1" gate="G$1" x="48.26" y="5.08" smashed="yes">
+<instance part="TV1" gate="G$1" x="48.26" y="5.08" smashed="yes">
 <attribute name="NAME" x="50.8" y="5.08" size="1.778" layer="95"/>
 <attribute name="VALUE" x="50.8" y="2.54" size="1.778" layer="96"/>
 </instance>
-<instance part="D3" gate="G$1" x="-38.1" y="2.54" smashed="yes">
+<instance part="LED1" gate="G$1" x="-38.1" y="2.54" smashed="yes">
 <attribute name="NAME" x="-34.544" y="-1.778" size="1.778" layer="95" rot="R90"/>
 <attribute name="VALUE" x="-32.385" y="-1.778" size="1.778" layer="96" rot="R90"/>
 </instance>
-<instance part="D4" gate="G$1" x="-38.1" y="-22.86" smashed="yes">
+<instance part="LED2" gate="G$1" x="-38.1" y="-22.86" smashed="yes">
 <attribute name="NAME" x="-34.544" y="-27.178" size="1.778" layer="95" rot="R90"/>
 <attribute name="VALUE" x="-32.385" y="-27.178" size="1.778" layer="96" rot="R90"/>
-</instance>
-<instance part="R3" gate="G$1" x="22.86" y="2.54" smashed="yes" rot="R180">
-<attribute name="VALUE" x="25.654" y="5.334" size="1.27" layer="96" rot="R180"/>
-<attribute name="NAME" x="25.908" y="0.508" size="1.27" layer="95" rot="R180"/>
 </instance>
 <instance part="RCS" gate="G$1" x="-22.86" y="40.64" smashed="yes" rot="R180">
@@
 <attribute name="NAME" x="-19.812" y="38.608" size="1.27" layer="95" rot="R180"/>
 </instance>
-<instance part="M2" gate="G$1" x="17.78" y="40.64" smashed="yes" rot="R90">
+<instance part="TV2" gate="G$1" x="17.78" y="40.64" smashed="yes" rot="R90">
 <attribute name="NAME" x="17.78" y="43.18" size="1.778" layer="95" rot="R90"/>
 <attribute name="VALUE" x="20.32" y="43.18" size="1.778" layer="96" rot="R90"/>
@@
 <attribute name="NAME" x="59.944" y="20.701" size="1.778" layer="95"/>
 <attribute name="VALUE" x="59.944" y="15.621" size="1.778" layer="96"/>
+</instance>
+<instance part="R4" gate="G$1" x="-38.1" y="12.7" smashed="yes" rot="R90">
+<attribute name="VALUE" x="-35.306" y="9.906" size="1.27" layer="96" rot="R90"/>
+<attribute name="NAME" x="-40.132" y="9.652" size="1.27" layer="95" rot="R90"/>
+</instance>
+<instance part="R5" gate="G$1" x="-38.1" y="-12.7" smashed="yes" rot="R90">
+<attribute name="VALUE" x="-35.306" y="-15.494" size="1.27" layer="96" rot="R90"/>
+<attribute name="NAME" x="-40.132" y="-15.748" size="1.27" layer="95" rot="R90"/>
+</instance>
+<instance part="R6" gate="G$1" x="22.86" y="2.54" smashed="yes" rot="R180">
+<attribute name="VALUE" x="25.654" y="5.334" size="1.27" layer="96" rot="R180"/>
+<attribute name="NAME" x="25.908" y="0.508" size="1.27" layer="95" rot="R180"/>
 </instance>
 </instances>
@@
 <wire x1="30.48" y1="35.56" x2="30.48" y2="40.64" width="0.1524" layer="91"/>
 <junction x="30.48" y="40.64"/>
-<pinref part="M2" gate="G$1" pin="D"/>
+<pinref part="TV2" gate="G$1" pin="D"/>
 </segment>
 </net>
@@
 <pinref part="L1" gate="G$1" pin="2"/>
 <wire x1="53.34" y1="40.64" x2="48.26" y2="40.64" width="0.1524" layer="91"/>
-<pinref part="M1" gate="G$1" pin="D"/>
+<pinref part="TV1" gate="G$1" pin="D"/>
 <wire x1="48.26" y1="40.64" x2="45.72" y2="40.64" width="0.1524" layer="91"/>
 <wire x1="48.26" y1="10.16" x2="48.26" y2="40.64" width="0.1524" layer="91"/>
@@
 <wire x1="48.26" y1="-30.48" x2="63.5" y2="-30.48" width="0.1524" layer="91"/>
 <label x="-48.26" y="-30.48" size="1.27" layer="95" rot="R180" xref="yes"/>
-<label x="66.04" y="-30.48" size="1.27" layer="95" xref="yes"/>
-<pinref part="M1" gate="G$1" pin="S"/>
-<wire x1="63.5" y1="-30.48" x2="66.04" y2="-30.48" width="0.1524" layer="91"/>
+<label x="78.74" y="-30.48" size="1.27" layer="95" xref="yes"/>
+<pinref part="TV1" gate="G$1" pin="S"/>
+<wire x1="63.5" y1="-30.48" x2="78.74" y2="-30.48" width="0.1524" layer="91"/>
 <wire x1="48.26" y1="0" x2="48.26" y2="-30.48" width="0.1524" layer="91"/>
 <junction x="48.26" y="-30.48"/>
@@
 <wire x1="0" y1="-30.48" x2="-38.1" y2="-30.48" width="0.1524" layer="91"/>
 <junction x="0" y="-30.48"/>
-<pinref part="D4" gate="G$1" pin="C"/>
+<pinref part="LED2" gate="G$1" pin="C"/>
 <wire x1="-38.1" y1="-30.48" x2="-48.26" y2="-30.48" width="0.1524" layer="91"/>
 <wire x1="-38.1" y1="-27.94" x2="-38.1" y2="-30.48" width="0.1524" layer="91"/>
@@
 <pinref part="DD1" gate="CN" pin="LDRV"/>
 <wire x1="12.7" y1="2.54" x2="17.78" y2="2.54" width="0.1524" layer="91"/>
-<pinref part="R3" gate="G$1" pin="P$2"/>
+<pinref part="R6" gate="G$1" pin="P$2"/>
 </segment>
 </net>
 <net name="N$9" class="0">
 <segment>
-<pinref part="M1" gate="G$1" pin="G"/>
+<pinref part="TV1" gate="G$1" pin="G"/>
 <wire x1="27.94" y1="2.54" x2="43.18" y2="2.54" width="0.1524" layer="91"/>
-<pinref part="R3" gate="G$1" pin="P$1"/>
+<pinref part="R6" gate="G$1" pin="P$1"/>
 </segment>
 </net>
@@
 <wire x1="12.7" y1="10.16" x2="15.24" y2="10.16" width="0.1524" layer="91"/>
 <wire x1="15.24" y1="10.16" x2="15.24" y2="35.56" width="0.1524" layer="91"/>
-<pinref part="M2" gate="G$1" pin="G"/>
+<pinref part="TV2" gate="G$1" pin="G"/>
 </segment>
 </net>
 <net name="N$1" class="0">
 <segment>
-<pinref part="D4" gate="G$1" pin="A"/>
-<pinref part="R2" gate="G$1" pin="P$1"/>
+<pinref part="LED2" gate="G$1" pin="A"/>
 <wire x1="-38.1" y1="-20.32" x2="-38.1" y2="-17.78" width="0.1524" layer="91"/>
+<pinref part="R5" gate="G$1" pin="P$1"/>
 </segment>
 </net>
 <net name="N$11" class="0">
 <segment>
-<pinref part="R2" gate="G$1" pin="P$2"/>
-<pinref part="D3" gate="G$1" pin="C"/>
+<pinref part="LED1" gate="G$1" pin="C"/>
 <wire x1="-38.1" y1="-7.62" x2="-38.1" y2="-5.08" width="0.1524" layer="91"/>
 <pinref part="DD1" gate="CN" pin="STAT"/>
@@
 <wire x1="-12.7" y1="-5.08" x2="-38.1" y2="-5.08" width="0.1524" layer="91"/>
 <junction x="-38.1" y="-5.08"/>
+<pinref part="R5" gate="G$1" pin="P$2"/>
 </segment>
 </net>
 <net name="N$12" class="0">
 <segment>
-<pinref part="D3" gate="G$1" pin="A"/>
-<pinref part="R1" gate="G$1" pin="P$1"/>
+<pinref part="LED1" gate="G$1" pin="A"/>
 <wire x1="-38.1" y1="5.08" x2="-38.1" y2="7.62" width="0.1524" layer="91"/>
+<pinref part="R4" gate="G$1" pin="P$1"/>
 </segment>
 </net>
@@
 <wire x1="12.7" y1="40.64" x2="-15.24" y2="40.64" width="0.1524" layer="91"/>
 <pinref part="RCS" gate="G$1" pin="P$1"/>
-<pinref part="M2" gate="G$1" pin="S"/>
+<pinref part="TV2" gate="G$1" pin="S"/>
 <wire x1="-15.24" y1="40.64" x2="-17.78" y2="40.64" width="0.1524" layer="91"/>
 <wire x1="-15.24" y1="10.16" x2="-15.24" y2="40.64" width="0.1524" layer="91"/>
@@
 <pinref part="C3" gate="G$1" pin="2"/>
 <wire x1="-33.02" y1="20.32" x2="-38.1" y2="20.32" width="0.1524" layer="91"/>
-<pinref part="R1" gate="G$1" pin="P$2"/>
 <wire x1="-38.1" y1="20.32" x2="-43.18" y2="20.32" width="0.1524" layer="91"/>
 <wire x1="-38.1" y1="17.78" x2="-38.1" y2="20.32" width="0.1524" layer="91"/>
 <junction x="-38.1" y="20.32"/>
-</segment>
-</net>
+<pinref part="R4" gate="G$1" pin="P$2"/>
+</segment>
+</net>

Commit message: Файлы обновлены
Parts:
- C0, C5, C6, C7: SPICEPREFIX (none) -> C
- R4, R5: value RESISTOR -> 45; device 1_RESISTOR:RESISTOR -> 1_RESISTOR:RESISTOR0603
- R6: device 1_RESISTOR:RESISTOR -> 1_RESISTOR:RESISTOR0603
- RCS: device 1_RESISTOR:RESISTOR0603 -> 1_RESISTOR:RESISTOR
- renumbered TV1 to VT1, TV2 to VT2
Connections:
- removed net N$15: C5.2, C6.1
- removed net N$16: C0.2, C7.1
- removed net N$3: C1.2, C4.1
- removed net N$7: C3.2, C4.2, R4.P$2
- net 8.4V: now also C6.1, C7.1
- net GND: now also C0.2, C1.2, C3.2, C4.2, C5.2
- net N$2: now also R4.P$2; no longer C3.1
- net V_IN: now also C3.1, C4.1
Other:
- moved on the sheet: C0, C1, C2, C3, C4, C5, C6, C7, LED1, LED2, R4, R5

Commit message: asd
Connections:
- removed net N$2: C2.2, R4.P$2
- net GND: now also C2.2
- net V_IN: now also R4.P$2
Changed lines of the file:
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@@
 <layer number="91" name="Nets" color="2" fill="1" visible="yes" active="yes"/>
 <layer number="92" name="Busses" color="1" fill="1" visible="yes" active="yes"/>
-<layer number="93" name="Pins" color="2" fill="1" visible="yes" active="yes"/>
+<layer number="93" name="Pins" color="2" fill="1" visible="no" active="yes"/>
 <layer number="94" name="Symbols" color="4" fill="1" visible="yes" active="yes"/>
 <layer number="95" name="Names" color="7" fill="1" visible="yes" active="yes"/>
@@
 <label x="-73.66" y="40.64" size="1.27" layer="95" rot="R180" xref="yes"/>
 <pinref part="DD1" gate="CN" pin="VIN"/>
-<wire x1="-30.48" y1="40.64" x2="-45.72" y2="40.64" width="0.1524" layer="91"/>
+<wire x1="-30.48" y1="40.64" x2="-38.1" y2="40.64" width="0.1524" layer="91"/>
+<wire x1="-38.1" y1="40.64" x2="-45.72" y2="40.64" width="0.1524" layer="91"/>
 <wire x1="-45.72" y1="40.64" x2="-53.34" y2="40.64" width="0.1524" layer="91"/>
 <wire x1="-53.34" y1="40.64" x2="-60.96" y2="40.64" width="0.1524" layer="91"/>
@@
 <wire x1="-45.72" y1="35.56" x2="-45.72" y2="40.64" width="0.1524" layer="91"/>
 <junction x="-45.72" y="40.64"/>
+<pinref part="R4" gate="G$1" pin="P$2"/>
+<wire x1="-45.72" y1="17.78" x2="-45.72" y2="20.32" width="0.1524" layer="91"/>
+<wire x1="-45.72" y1="20.32" x2="-38.1" y2="20.32" width="0.1524" layer="91"/>
+<wire x1="-38.1" y1="20.32" x2="-38.1" y2="40.64" width="0.1524" layer="91"/>
+<junction x="-38.1" y="40.64"/>
 </segment>
 </net>
@@
 <wire x1="0" y1="-30.48" x2="-45.72" y2="-30.48" width="0.1524" layer="91"/>
 <junction x="0" y="-30.48"/>
-<wire x1="-45.72" y1="-30.48" x2="-53.34" y2="-30.48" width="0.1524" layer="91"/>
+<wire x1="-45.72" y1="-30.48" x2="-50.8" y2="-30.48" width="0.1524" layer="91"/>
+<wire x1="-50.8" y1="-30.48" x2="-53.34" y2="-30.48" width="0.1524" layer="91"/>
 <wire x1="-53.34" y1="-30.48" x2="-60.96" y2="-30.48" width="0.1524" layer="91"/>
 <wire x1="-60.96" y1="-30.48" x2="-68.58" y2="-30.48" width="0.1524" layer="91"/>
@@
 <wire x1="-45.72" y1="-27.94" x2="-45.72" y2="-30.48" width="0.1524" layer="91"/>
 <junction x="-45.72" y="-30.48"/>
-<pinref part="C1" gate="G$1" pin="2"/>
-<wire x1="-53.34" y1="27.94" x2="-53.34" y2="-30.48" width="0.1524" layer="91"/>
 <pinref part="C4" gate="G$1" pin="2"/>
 <wire x1="-60.96" y1="27.94" x2="-60.96" y2="-30.48" width="0.1524" layer="91"/>
@@
 <wire x1="91.44" y1="27.94" x2="91.44" y2="-30.48" width="0.1524" layer="91"/>
 <junction x="91.44" y="-30.48"/>
+<pinref part="C2" gate="G$1" pin="2"/>
+<wire x1="-45.72" y1="27.94" x2="-45.72" y2="25.4" width="0.1524" layer="91"/>
+<wire x1="-45.72" y1="25.4" x2="-50.8" y2="25.4" width="0.1524" layer="91"/>
+<wire x1="-50.8" y1="25.4" x2="-50.8" y2="-30.48" width="0.1524" layer="91"/>
+<junction x="-50.8" y="-30.48"/>
+<pinref part="C1" gate="G$1" pin="2"/>
+<wire x1="-53.34" y1="27.94" x2="-53.34" y2="-30.48" width="0.1524" layer="91"/>
+<junction x="-53.34" y="-30.48"/>
 </segment>
 </net>
@@
 </segment>
 </net>
-<net name="N$2" class="0">
-<segment>
-<pinref part="C2" gate="G$1" pin="2"/>
-<pinref part="R4" gate="G$1" pin="P$2"/>
-<wire x1="-45.72" y1="27.94" x2="-45.72" y2="17.78" width="0.1524" layer="91"/>
-</segment>
-</net>
