File: shema.brd (EAGLE design)
At the start: 100 x 80 mm, 14 parts, among them M1 TRANSISTORN, M2 TRAN_P

Commit message: Файлы обновлены
Parts:
- removed D3, D4: LED, 1_LED:1206
- removed M1: TRANSISTORN, 1_TRANSISTOR (2):PDFN5*6-8L
- removed M2: TRAN_P, 1_TRANSISTOR (2):SOP-8
- removed R1, R2: RESISTOR0603, 1_RESISTOR:0603
- removed R3: 1.8, 1_RESISTOR:0603
- added C2, C3, C4, C5, C6, C7: 22uF, 1_RESISTOR:1206
- added LED1, LED2: LED, 1_LED:1206
- added R4, R5: 45, 1_RESISTOR:0603
- added R6: 1.8, 1_RESISTOR:0603
- added VT1: TRANSISTORN, 1_TRANSISTOR (2):PDFN5*6-8L
- added VT2: TRAN_P, 1_TRANSISTOR (2):SOP-8
- moved C0 79.5 mm to (45.2, 25.9), turned to 270 degrees
- moved D1 66.2 mm to (44.0, 33.3)
- moved L1 63.6 mm to (35.1, 33.4)
- moved RCS 57.2 mm to (20.0, 33.0), turned to 180 degrees
- moved D2 55.0 mm to (24.5, 18.8)
- moved C1 47.3 mm to (7.76, 37.0)
- moved DD1 31.7 mm to (15.1, 25.7)
Connections:
- new net N$2: C2.P$2, R4.P$2
- net 8.4V: now also C5.P$1, C6.P$1, C7.P$1
- net GND: now also C3.P$2, C4.P$2, C5.P$2, C6.P$2, C7.P$2, LED2.C, VT1.P$5, VT1.P$6, VT1.P$7; no longer D4.C, M1.P$5, M1.P$6, M1.P$7
- net N$1: now also LED2.A, R5.P$1; no longer D4.A, R2.P$1
- net N$10: now also VT2.P$4; no longer M2.P$4
- net N$11: now also LED1.C, R5.P$2; no longer D3.C, R2.P$2
- net N$12: now also LED1.A, R4.P$1; no longer D3.A, R1.P$1
- net N$4: now also VT2.P$1, VT2.P$2, VT2.P$3; no longer M2.P$1, M2.P$2, M2.P$3
- net N$5: now also VT2.P$5, VT2.P$6, VT2.P$7, VT2.P$8; no longer M2.P$5, M2.P$6, M2.P$7, M2.P$8
- net N$6: now also VT1.P$1, VT1.P$2, VT1.P$3, VT1.P$4, VT1.P$9; no longer M1.P$1, M1.P$2, M1.P$3, M1.P$4, M1.P$9
- net N$8: now also R6.P$2; no longer R3.P$2
- net N$9: now also R6.P$1, VT1.P$8; no longer M1.P$8, R3.P$1
- net V_IN: now also C2.P$1, C3.P$1, C4.P$1; no longer R1.P$2

Commit message: asd
Connections:
- removed net N$2: C2.P$2, R4.P$2
- net GND: now also C2.P$2
- net V_IN: now also R4.P$2
Changed lines of the file:
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@@
 <contactref element="C1" pad="P$1"/>
 <contactref element="C2" pad="P$1"/>
-<wire x1="6.526" y1="37.02" x2="17.15" y2="33" width="0" layer="19" extent="1-1"/>
-<wire x1="9.094" y1="34.98" x2="6.526" y2="37.02" width="0" layer="19" extent="1-1"/>
-<wire x1="10.776" y1="34.75" x2="9.094" y2="34.98" width="0" layer="19" extent="1-1"/>
+<contactref element="R4" pad="P$2"/>
+<wire x1="14.505" y1="28.07" x2="17.15" y2="33" width="0" layer="19" extent="1-1"/>
+<wire x1="14.505" y1="23.27" x2="14.505" y2="28.07" width="0" layer="19" extent="1-1"/>
+<wire x1="9.95" y1="31.218" x2="14.505" y2="28.07" width="0" layer="19" extent="1-1"/>
+<wire x1="10.776" y1="34.75" x2="9.95" y2="31.218" width="0" layer="19" extent="1-1"/>
+<wire x1="9.094" y1="34.98" x2="10.776" y2="34.75" width="0" layer="19" extent="1-1"/>
 <wire x1="10.716" y1="37.02" x2="10.776" y2="34.75" width="0" layer="19" extent="1-1"/>
-<wire x1="14.505" y1="28.07" x2="10.776" y2="34.75" width="0" layer="19" extent="1-1"/>
-<wire x1="14.505" y1="23.27" x2="14.505" y2="28.07" width="0" layer="19" extent="1-1"/>
+<wire x1="6.526" y1="37.02" x2="9.094" y2="34.98" width="0" layer="19" extent="1-1"/>
 </signal>
 <signal name="N$5">
@@
 <contactref element="D2" pad="A"/>
 <contactref element="LED2" pad="C"/>
-<contactref element="C1" pad="P$2"/>
 <contactref element="C4" pad="P$2"/>
 <contactref element="C3" pad="P$2"/>
@@
 <contactref element="C7" pad="P$2"/>
 <contactref element="C6" pad="P$2"/>
+<contactref element="C2" pad="P$2"/>
+<contactref element="C1" pad="P$2"/>
 <wire x1="42.75" y1="24.669" x2="45.19" y2="24.609" width="0" layer="19" extent="1-1"/>
 <wire x1="45.29" y1="20.639" x2="45.19" y2="24.609" width="0" layer="19" extent="1-1"/>
-<wire x1="42.94" y1="20.669" x2="42.75" y2="24.669" width="0" layer="19" extent="1-1"/>
-<wire x1="27.019" y1="28.57" x2="42.94" y2="20.669" width="0" layer="19" extent="1-1"/>
+<wire x1="42.94" y1="20.669" x2="45.29" y2="20.639" width="0" layer="19" extent="1-1"/>
+<wire x1="27.019" y1="28.57" x2="42.75" y2="24.669" width="0" layer="19" extent="1-1"/>
 <wire x1="25.79" y1="28.57" x2="27.019" y2="28.57" width="0" layer="19" extent="1-1"/>
 <wire x1="24.465" y1="28.57" x2="25.79" y2="28.57" width="0" layer="19" extent="1-1"/>
 <wire x1="17.045" y1="23.27" x2="24.465" y2="28.57" width="0" layer="19" extent="1-1"/>
-<wire x1="13.251" y1="34.75" x2="17.045" y2="23.27" width="0" layer="19" extent="1-1"/>
-<wire x1="9.001" y1="37.02" x2="13.251" y2="34.75" width="0" layer="19" extent="1-1"/>
-<wire x1="6.619" y1="34.98" x2="9.001" y2="37.02" width="0" layer="19" extent="1-1"/>
 <wire x1="21.215" y1="18.78" x2="17.045" y2="23.27" width="0" layer="19" extent="1-1"/>
 <wire x1="9.92" y1="20.862" x2="17.045" y2="23.27" width="0" layer="19" extent="1-1"/>
+<wire x1="13.251" y1="34.75" x2="17.045" y2="23.27" width="0" layer="19" extent="1-1"/>
+<wire x1="13.191" y1="37.02" x2="13.251" y2="34.75" width="0" layer="19" extent="1-1"/>
+<wire x1="9.001" y1="37.02" x2="13.191" y2="37.02" width="0" layer="19" extent="1-1"/>
+<wire x1="6.619" y1="34.98" x2="9.001" y2="37.02" width="0" layer="19" extent="1-1"/>
 </signal>
 <signal name="N$8">
@@
 <wire x1="13.235" y1="28.07" x2="26.735" y2="30.62" width="0" layer="19" extent="1-1"/>
 </signal>
-<signal name="N$2">
-<contactref element="C2" pad="P$2"/>
-<contactref element="R4" pad="P$2"/>
-<wire x1="9.95" y1="31.218" x2="13.191" y2="37.02" width="0" layer="19" extent="1-1"/>
-</signal>
 </signals>
