File: shema.brd (EAGLE design)
At the start: 100 x 80 mm, 20 parts

Commit message: изменения файлов
Parts:
- moved C0 63.0 mm to (-17.8, 24.9)
- moved C5 63.0 mm to (-20.2, 24.9)
- moved C6 63.0 mm to (-20.1, 20.9)
- moved C7 63.0 mm to (-17.7, 20.9)
- moved D1 58.0 mm to (-14.0, 31.3)
- moved L1 58.0 mm to (-22.9, 31.4)
- moved VT2 57.0 mm to (-29.6, 31.2)
- moved RCS 56.0 mm to (-36.0, 31.0)
- moved C1 54.2 mm to (-46.2, 32.0)
- moved C2 54.2 mm to (-42.0, 32.0)
- moved C3 54.2 mm to (-46.1, 30.0)
- moved C4 54.2 mm to (-42.0, 29.8)
- moved LED2 53.2 mm to (-43.1, 23.4)
- moved D2 51.1 mm to (-26.5, 15.8)
- moved R5 50.9 mm to (-40.8, 20.0), turned to 0 degrees
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
Commit message: изменение файлов
Parts:
- moved D2 70.9 mm to (44.2, 20.5), turned to 90 degrees
- moved C6 61.9 mm to (41.1, 11.1), turned to 90 degrees
- moved C3 59.1 mm to (10.8, 14.1), turned to 270 degrees
- moved C4 57.2 mm to (13.0, 14.0), turned to 270 degrees
- moved C7 56.6 mm to (38.0, 11.2), turned to 90 degrees
- moved C0 54.4 mm to (34.8, 11.2), turned to 90 degrees
- moved C5 54.3 mm to (32.2, 11.1), turned to 90 degrees
- moved C1 54.2 mm to (4.91, 14.1), turned to 270 degrees
- moved C2 53.6 mm to (8.46, 14.0), turned to 270 degrees
- moved R6 53.6 mm to (22.3, 10.8), turned to 180 degrees
- moved DD1 52.9 mm to (17.2, 13.1), turned to 270 degrees
- moved VT1 52.8 mm to (26.8, 12.2), turned to 90 degrees
- moved VT2 52.3 mm to (21.5, 20.3), turned to 0 degrees
- moved L1 52.3 mm to (28.4, 20.9), turned to 270 degrees
- moved RCS 52.0 mm to (14.4, 18.4)
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
Commit message: изменение файлов
Parts:
- moved C4 10.4 mm to (3.03, 11.0), turned to 180 degrees
- moved C3 7.67 mm to (3.12, 14.2), turned to 180 degrees
- moved C2 6.48 mm to (3.02, 17.5), turned to 180 degrees
- moved C1 6.27 mm to (3.09, 20.1), turned to 180 degrees
- moved C7 6.06 mm to (32.0, 10.8), turned to 270 degrees
- moved C5 5.50 mm to (37.8, 10.9), turned to 270 degrees
- moved LED2 5.39 mm to (7.70, 11.8)
- moved R5 5.39 mm to (7.57, 15.7)
- moved DD1 4.12 mm to (13.2, 12.1)
- moved R4 4.05 mm to (6.70, 20.0), turned to 90 degrees
- moved D2 3.34 mm to (40.9, 20.0)
- moved R6 3.00 mm to (19.3, 10.8)
- moved VT2 2.84 mm to (18.7, 20.7)
- moved D1 2.76 mm to (33.8, 18.8)
- moved RCS 2.74 mm to (12.6, 20.4), turned to 270 degrees
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
Commit message: файлы изменения
Parts:
- moved D1 1.00 mm to (33.8, 19.8)
- moved VT2 0.58 mm to (18.7, 21.3), turned to 270 degrees
- moved RCS 0.17 mm to (12.4, 20.6), turned to 90 degrees
Changed lines of the file:
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@@
 <attribute name="VALUE" x="30.657" y="12.3" size="0.4064" layer="27" rot="R270"/>
 </element>
-<element name="D1" library="1_DIOD" package="CB417-15" value="B560C-13-F" x="33.83" y="18.8" smashed="yes" rot="R270">
-<attribute name="NAME" x="37.132" y="22.356" size="1.27" layer="25" rot="R270"/>
-<attribute name="VALUE" x="29.258" y="22.229" size="1.27" layer="27" rot="R270"/>
+<element name="D1" library="1_DIOD" package="CB417-15" value="B560C-13-F" x="33.83" y="19.8" smashed="yes" rot="R270">
+<attribute name="NAME" x="37.132" y="23.356" size="1.27" layer="25" rot="R270"/>
+<attribute name="VALUE" x="29.258" y="23.229" size="1.27" layer="27" rot="R270"/>
 </element>
 <element name="D2" library="1_DIOD" package="DIOD" value="SS36C" x="40.93" y="19.97" smashed="yes" rot="R90">
@@
 <attribute name="VALUE" x="20.327" y="11.937" size="0.4064" layer="27" rot="R180"/>
 </element>
-<element name="RCS" library="1_RESISTOR" package="2512" value="0.015" x="12.56" y="20.44" smashed="yes" rot="R270">
-<attribute name="NAME" x="14.719" y="23.488" size="1.016" layer="25" rot="R270"/>
-<attribute name="VALUE" x="9.766" y="23.615" size="1.016" layer="27" rot="R270"/>
+<element name="RCS" library="1_RESISTOR" package="2512" value="0.015" x="12.44" y="20.56" smashed="yes" rot="R90">
+<attribute name="NAME" x="10.281" y="17.512" size="1.016" layer="25" rot="R90"/>
+<attribute name="VALUE" x="15.234" y="17.385" size="1.016" layer="27" rot="R90"/>
 </element>
 <element name="VT1" library="1_TRANSISTOR (2)" package="PDFN5*6-8L" value="TRANSISTORN" x="25.21" y="12.16" smashed="yes">
@@
 <attribute name="VALUE" x="22.285" y="10.162" size="1.27" layer="27" rot="R90"/>
 </element>
-<element name="VT2" library="1_TRANSISTOR (2)" package="SOP-8" value="TRAN_P" x="18.71" y="20.71" smashed="yes">
-<attribute name="NAME" x="15.662" y="24.012" size="1.27" layer="25"/>
-<attribute name="VALUE" x="15.535" y="16.265" size="1.27" layer="27"/>
+<element name="VT2" library="1_TRANSISTOR (2)" package="SOP-8" value="TRAN_P" x="18.71" y="21.29" smashed="yes" rot="R270">
+<attribute name="NAME" x="22.012" y="24.338" size="1.27" layer="25" rot="R270"/>
+<attribute name="VALUE" x="14.265" y="24.465" size="1.27" layer="27" rot="R270"/>
 </element>
 </elements>
@@
 <contactref element="R4" pad="P$2"/>
 <wire x1="10.82" y1="12.765" x2="15.62" y2="12.765" width="0" layer="19" extent="1-1"/>
-<wire x1="12.56" y1="17.59" x2="10.82" y2="12.765" width="0" layer="19" extent="1-1"/>
-<wire x1="6.7" y1="20.658" x2="12.56" y2="17.59" width="0" layer="19" extent="1-1"/>
+<wire x1="12.44" y1="23.41" x2="10.82" y2="12.765" width="0" layer="19" extent="1-1"/>
+<wire x1="6.7" y1="20.658" x2="12.44" y2="23.41" width="0" layer="19" extent="1-1"/>
 <wire x1="4.324" y1="20.09" x2="6.7" y2="20.658" width="0" layer="19" extent="1-1"/>
 <wire x1="4.254" y1="17.54" x2="4.324" y2="20.09" width="0" layer="19" extent="1-1"/>
@@
 <contactref element="VT2" pad="P$8"/>
 <wire x1="26.35" y1="23.66" x2="40.93" y2="23.275" width="0" layer="19" extent="1-1"/>
-<wire x1="20.615" y1="18.11" x2="26.35" y2="23.66" width="0" layer="19" extent="1-1"/>
-<wire x1="19.345" y1="18.11" x2="20.615" y2="18.11" width="0" layer="19" extent="1-1"/>
-<wire x1="18.075" y1="18.11" x2="19.345" y2="18.11" width="0" layer="19" extent="1-1"/>
-<wire x1="16.805" y1="18.11" x2="18.075" y2="18.11" width="0" layer="19" extent="1-1"/>
+<wire x1="16.11" y1="19.385" x2="26.35" y2="23.66" width="0" layer="19" extent="1-1"/>
+<wire x1="16.11" y1="20.655" x2="16.11" y2="19.385" width="0" layer="19" extent="1-1"/>
+<wire x1="16.11" y1="21.925" x2="16.11" y2="20.655" width="0" layer="19" extent="1-1"/>
+<wire x1="16.11" y1="23.195" x2="16.11" y2="21.925" width="0" layer="19" extent="1-1"/>
 </signal>
 <signal name="N$6">
@@
 <contactref element="VT1" pad="P$4"/>
 <contactref element="VT1" pad="P$9"/>
-<wire x1="26.35" y1="18.06" x2="33.83" y2="22.179" width="0" layer="19" extent="1-1"/>
+<wire x1="26.35" y1="18.06" x2="33.83" y2="23.179" width="0" layer="19" extent="1-1"/>
 <wire x1="25.845" y1="14.81" x2="26.35" y2="18.06" width="0" layer="19" extent="1-1"/>
 <wire x1="27.115" y1="14.81" x2="25.845" y2="14.81" width="0" layer="19" extent="1-1"/>
@@
 <contactref element="DD1" pad="6"/>
 <contactref element="VT2" pad="P$4"/>
-<wire x1="15.62" y1="11.495" x2="20.615" y2="23.31" width="0" layer="19" extent="1-1"/>
+<wire x1="15.62" y1="11.495" x2="21.31" y2="19.385" width="0" layer="19" extent="1-1"/>
 </signal>
 <signal name="N$1">
@@
 <wire x1="35.19" y1="12.084" x2="37.75" y2="12.144" width="0" layer="19" extent="1-1"/>
 <wire x1="31.98" y1="12.014" x2="35.19" y2="12.084" width="0" layer="19" extent="1-1"/>
-<wire x1="33.83" y1="15.445" x2="35.19" y2="12.084" width="0" layer="19" extent="1-1"/>
+<wire x1="33.83" y1="16.445" x2="35.19" y2="12.084" width="0" layer="19" extent="1-1"/>
 <wire x1="10.82" y1="11.495" x2="31.98" y2="12.014" width="0" layer="19" extent="1-1"/>
 </signal>
@@
 <contactref element="VT2" pad="P$2"/>
 <contactref element="VT2" pad="P$3"/>
-<wire x1="19.345" y1="23.31" x2="18.075" y2="23.31" width="0" layer="19" extent="1-1"/>
-<wire x1="16.805" y1="23.31" x2="18.075" y2="23.31" width="0" layer="19" extent="1-1"/>
-<wire x1="12.56" y1="23.29" x2="16.805" y2="23.31" width="0" layer="19" extent="1-1"/>
-<wire x1="15.62" y1="14.035" x2="16.805" y2="23.31" width="0" layer="19" extent="1-1"/>
+<wire x1="21.31" y1="20.655" x2="21.31" y2="21.925" width="0" layer="19" extent="1-1"/>
+<wire x1="21.31" y1="23.195" x2="21.31" y2="21.925" width="0" layer="19" extent="1-1"/>
+<wire x1="12.44" y1="17.71" x2="21.31" y2="23.195" width="0" layer="19" extent="1-1"/>
+<wire x1="15.62" y1="14.035" x2="21.31" y2="23.195" width="0" layer="19" extent="1-1"/>
 </signal>
 </signals>

Commit message: файлы изменения
Parts:
- moved C7 13.7 mm to (33.9, 24.4), turned to 0 degrees
- moved D2 13.6 mm to (27.6, 22.6), turned to 180 degrees
- moved C5 13.5 mm to (37.7, 24.4), turned to 0 degrees
- moved C6 11.4 mm to (37.8, 21.9), turned to 0 degrees
- moved C0 11.0 mm to (33.9, 21.7), turned to 0 degrees
- moved L1 7.62 mm to (19.4, 23.9)
- moved D1 6.00 mm to (33.1, 13.8)
- moved RCS 4.16 mm to (9.44, 23.4), turned to 180 degrees
- moved VT2 4.00 mm to (18.7, 17.3)
- moved R6 1.33 mm to (18.0, 10.5)
- moved VT1 1.09 mm to (25.8, 13.1)
- moved DD1 0.43 mm to (12.8, 12.3)

Commit message: файлы изменения
Parts:
- moved C5 1.07 mm to (38.3, 23.6), turned to 180 degrees
- moved C6 0.87 mm to (38.2, 21.1), turned to 180 degrees
- moved C7 0.82 mm to (34.1, 23.6), turned to 180 degrees
- moved C0 0.55 mm to (34.1, 21.3), turned to 180 degrees
Changed lines of the file:
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@@
 </autorouter>
 <elements>
-<element name="C0" library="1_RESISTOR" package="1206" value="22uF" x="33.85" y="21.73" smashed="yes">
-<attribute name="NAME" x="32.495" y="22.785" size="0.4064" layer="25"/>
-<attribute name="SPICEPREFIX" value="C" x="33.85" y="21.73" size="1.778" layer="27" display="off"/>
-<attribute name="VALUE" x="32.33" y="20.407" size="0.4064" layer="27"/>
+<element name="C0" library="1_RESISTOR" package="1206" value="22uF" x="34.15" y="21.27" smashed="yes" rot="R180">
+<attribute name="NAME" x="35.505" y="20.215" size="0.4064" layer="25" rot="R180"/>
+<attribute name="SPICEPREFIX" value="C" x="34.15" y="21.27" size="1.778" layer="27" rot="R180" display="off"/>
+<attribute name="VALUE" x="35.67" y="22.593" size="0.4064" layer="27" rot="R180"/>
 </element>
 <element name="C1" library="1_RESISTOR" package="1206" value="22uF" x="3.09" y="20.09" smashed="yes" rot="R180">
@@
 <attribute name="VALUE" x="4.55" y="12.303" size="0.4064" layer="27" rot="R180"/>
 </element>
-<element name="C5" library="1_RESISTOR" package="1206" value="22uF" x="37.71" y="24.45" smashed="yes">
-<attribute name="NAME" x="36.355" y="25.505" size="0.4064" layer="25"/>
-<attribute name="SPICEPREFIX" value="C" x="37.71" y="24.45" size="1.778" layer="27" display="off"/>
-<attribute name="VALUE" x="36.19" y="23.127" size="0.4064" layer="27"/>
-</element>
-<element name="C6" library="1_RESISTOR" package="1206" value="22uF" x="37.83" y="21.9" smashed="yes">
-<attribute name="NAME" x="36.475" y="22.955" size="0.4064" layer="25"/>
-<attribute name="SPICEPREFIX" value="C" x="37.83" y="21.9" size="1.778" layer="27" display="off"/>
-<attribute name="VALUE" x="36.31" y="20.577" size="0.4064" layer="27"/>
-</element>
-<element name="C7" library="1_RESISTOR" package="1206" value="22uF" x="33.88" y="24.39" smashed="yes">
-<attribute name="NAME" x="32.525" y="25.445" size="0.4064" layer="25"/>
-<attribute name="SPICEPREFIX" value="C" x="33.88" y="24.39" size="1.778" layer="27" display="off"/>
-<attribute name="VALUE" x="32.36" y="23.067" size="0.4064" layer="27"/>
+<element name="C5" library="1_RESISTOR" package="1206" value="22uF" x="38.29" y="23.55" smashed="yes" rot="R180">
+<attribute name="NAME" x="39.645" y="22.495" size="0.4064" layer="25" rot="R180"/>
+<attribute name="SPICEPREFIX" value="C" x="38.29" y="23.55" size="1.778" layer="27" rot="R180" display="off"/>
+<attribute name="VALUE" x="39.81" y="24.873" size="0.4064" layer="27" rot="R180"/>
+</element>
+<element name="C6" library="1_RESISTOR" package="1206" value="22uF" x="38.17" y="21.1" smashed="yes" rot="R180">
+<attribute name="NAME" x="39.525" y="20.045" size="0.4064" layer="25" rot="R180"/>
+<attribute name="SPICEPREFIX" value="C" x="38.17" y="21.1" size="1.778" layer="27" rot="R180" display="off"/>
+<attribute name="VALUE" x="39.69" y="22.423" size="0.4064" layer="27" rot="R180"/>
+</element>
+<element name="C7" library="1_RESISTOR" package="1206" value="22uF" x="34.12" y="23.61" smashed="yes" rot="R180">
+<attribute name="NAME" x="35.475" y="22.555" size="0.4064" layer="25" rot="R180"/>
+<attribute name="SPICEPREFIX" value="C" x="34.12" y="23.61" size="1.778" layer="27" rot="R180" display="off"/>
+<attribute name="VALUE" x="35.64" y="24.933" size="0.4064" layer="27" rot="R180"/>
 </element>
 <element name="D1" library="1_DIOD" package="CB417-15" value="B560C-13-F" x="33.08" y="13.85" smashed="yes" rot="R270">
@@
 <contactref element="C3" pad="P$2"/>
 <contactref element="C4" pad="P$2"/>
-<wire x1="39.071" y1="21.9" x2="38.951" y2="24.45" width="0" layer="19" extent="1-1"/>
-<wire x1="35.121" y1="24.39" x2="38.951" y2="24.45" width="0" layer="19" extent="1-1"/>
-<wire x1="35.091" y1="21.73" x2="35.121" y2="24.39" width="0" layer="19" extent="1-1"/>
-<wire x1="30.865" y1="22.62" x2="35.091" y2="21.73" width="0" layer="19" extent="1-1"/>
+<wire x1="36.929" y1="21.1" x2="37.049" y2="23.55" width="0" layer="19" extent="1-1"/>
+<wire x1="32.879" y1="23.61" x2="37.049" y2="23.55" width="0" layer="19" extent="1-1"/>
+<wire x1="32.909" y1="21.27" x2="32.879" y2="23.61" width="0" layer="19" extent="1-1"/>
+<wire x1="30.865" y1="22.62" x2="32.909" y2="21.27" width="0" layer="19" extent="1-1"/>
 <wire x1="26.405" y1="10.45" x2="30.865" y2="22.62" width="0" layer="19" extent="1-1"/>
 <wire x1="25.08" y1="10.45" x2="26.405" y2="10.45" width="0" layer="19" extent="1-1"/>
@@
 <contactref element="C7" pad="P$1"/>
 <contactref element="C6" pad="P$1"/>
-<wire x1="36.596" y1="21.9" x2="36.476" y2="24.45" width="0" layer="19" extent="1-1"/>
-<wire x1="32.646" y1="24.39" x2="36.476" y2="24.45" width="0" layer="19" extent="1-1"/>
-<wire x1="32.616" y1="21.73" x2="32.646" y2="24.39" width="0" layer="19" extent="1-1"/>
-<wire x1="33.08" y1="10.495" x2="32.616" y2="21.73" width="0" layer="19" extent="1-1"/>
+<wire x1="39.404" y1="21.1" x2="39.524" y2="23.55" width="0" layer="19" extent="1-1"/>
+<wire x1="35.354" y1="23.61" x2="39.524" y2="23.55" width="0" layer="19" extent="1-1"/>
+<wire x1="35.384" y1="21.27" x2="35.354" y2="23.61" width="0" layer="19" extent="1-1"/>
+<wire x1="33.08" y1="10.495" x2="35.384" y2="21.27" width="0" layer="19" extent="1-1"/>
 <wire x1="10.45" y1="11.705" x2="33.08" y2="10.495" width="0" layer="19" extent="1-1"/>
 </signal>

Commit message: файлы изменения
Parts:
- moved R6 6.08 mm to (24.0, 9.47)
- moved VT2 4.47 mm to (20.7, 13.3)
- moved L1 4.12 mm to (20.4, 19.9)
- moved RCS 3.61 mm to (11.4, 20.4)
- moved D1 3.16 mm to (36.1, 12.8)
- moved VT1 3.00 mm to (28.8, 13.1)
- moved D2 2.24 mm to (28.6, 20.6)
- moved C0 1.41 mm to (35.1, 20.3)
- moved C5 1.41 mm to (39.3, 22.6)
- moved C6 1.41 mm to (39.2, 20.1)
- moved C7 1.41 mm to (35.1, 22.6)
