File: shema.brd (EAGLE design)
At the start: 100 x 80 mm, 20 parts

Commit message: изменения файлов
Parts:
- moved D2 10.1 mm to (35.6, 13.4), turned to 90 degrees
- moved D1 8.06 mm to (44.1, 13.8)
- moved C7 7.12 mm to (41.9, 20.4), turned to 0 degrees
- moved C5 6.13 mm to (33.6, 20.3), turned to 0 degrees
- moved C0 5.81 mm to (29.3, 20.2), turned to 0 degrees
- moved C6 1.78 mm to (37.4, 20.4), turned to 0 degrees
Changed lines of the file:
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@@
 </autorouter>
 <elements>
-<element name="C0" library="1_RESISTOR" package="1206" value="22uF" x="35.15" y="20.27" smashed="yes" rot="R180">
-<attribute name="NAME" x="36.505" y="19.215" size="0.4064" layer="25" rot="R180"/>
-<attribute name="SPICEPREFIX" value="C" x="35.15" y="20.27" size="1.778" layer="27" rot="R180" display="off"/>
-<attribute name="VALUE" x="36.67" y="21.593" size="0.4064" layer="27" rot="R180"/>
+<element name="C0" library="1_RESISTOR" package="1206" value="22uF" x="29.34" y="20.2" smashed="yes">
+<attribute name="NAME" x="27.985" y="21.255" size="0.4064" layer="25"/>
+<attribute name="SPICEPREFIX" value="C" x="29.34" y="20.2" size="1.778" layer="27" display="off"/>
+<attribute name="VALUE" x="27.82" y="18.877" size="0.4064" layer="27"/>
 </element>
 <element name="C1" library="1_RESISTOR" package="1206" value="22uF" x="3.09" y="20.09" smashed="yes" rot="R180">
@@
 <attribute name="VALUE" x="4.55" y="12.303" size="0.4064" layer="27" rot="R180"/>
 </element>
-<element name="C5" library="1_RESISTOR" package="1206" value="22uF" x="39.29" y="22.55" smashed="yes" rot="R180">
-<attribute name="NAME" x="40.645" y="21.495" size="0.4064" layer="25" rot="R180"/>
-<attribute name="SPICEPREFIX" value="C" x="39.29" y="22.55" size="1.778" layer="27" rot="R180" display="off"/>
-<attribute name="VALUE" x="40.81" y="23.873" size="0.4064" layer="27" rot="R180"/>
-</element>
-<element name="C6" library="1_RESISTOR" package="1206" value="22uF" x="39.17" y="20.1" smashed="yes" rot="R180">
-<attribute name="NAME" x="40.525" y="19.045" size="0.4064" layer="25" rot="R180"/>
-<attribute name="SPICEPREFIX" value="C" x="39.17" y="20.1" size="1.778" layer="27" rot="R180" display="off"/>
-<attribute name="VALUE" x="40.69" y="21.423" size="0.4064" layer="27" rot="R180"/>
-</element>
-<element name="C7" library="1_RESISTOR" package="1206" value="22uF" x="35.12" y="22.61" smashed="yes" rot="R180">
-<attribute name="NAME" x="36.475" y="21.555" size="0.4064" layer="25" rot="R180"/>
-<attribute name="SPICEPREFIX" value="C" x="35.12" y="22.61" size="1.778" layer="27" rot="R180" display="off"/>
-<attribute name="VALUE" x="36.64" y="23.933" size="0.4064" layer="27" rot="R180"/>
-</element>
-<element name="D1" library="1_DIOD" package="CB417-15" value="B560C-13-F" x="36.08" y="12.85" smashed="yes" rot="R270">
-<attribute name="NAME" x="39.382" y="16.406" size="1.27" layer="25" rot="R270"/>
-<attribute name="VALUE" x="31.508" y="16.279" size="1.27" layer="27" rot="R270"/>
-</element>
-<element name="D2" library="1_DIOD" package="DIOD" value="SS36C" x="28.56" y="20.62" smashed="yes" rot="R180">
-<attribute name="NAME" x="32.255" y="17.349" size="1.27" layer="25" rot="R180"/>
-<attribute name="VALUE" x="32.046" y="25.109" size="1.27" layer="27" rot="R180"/>
+<element name="C5" library="1_RESISTOR" package="1206" value="22uF" x="33.58" y="20.33" smashed="yes">
+<attribute name="NAME" x="32.225" y="21.385" size="0.4064" layer="25"/>
+<attribute name="SPICEPREFIX" value="C" x="33.58" y="20.33" size="1.778" layer="27" display="off"/>
+<attribute name="VALUE" x="32.06" y="19.007" size="0.4064" layer="27"/>
+</element>
+<element name="C6" library="1_RESISTOR" package="1206" value="22uF" x="37.42" y="20.45" smashed="yes">
+<attribute name="NAME" x="36.065" y="21.505" size="0.4064" layer="25"/>
+<attribute name="SPICEPREFIX" value="C" x="37.42" y="20.45" size="1.778" layer="27" display="off"/>
+<attribute name="VALUE" x="35.9" y="19.127" size="0.4064" layer="27"/>
+</element>
+<element name="C7" library="1_RESISTOR" package="1206" value="22uF" x="41.88" y="20.39" smashed="yes">
+<attribute name="NAME" x="40.525" y="21.445" size="0.4064" layer="25"/>
+<attribute name="SPICEPREFIX" value="C" x="41.88" y="20.39" size="1.778" layer="27" display="off"/>
+<attribute name="VALUE" x="40.36" y="19.067" size="0.4064" layer="27"/>
+</element>
+<element name="D1" library="1_DIOD" package="CB417-15" value="B560C-13-F" x="44.08" y="13.85" smashed="yes" rot="R270">
+<attribute name="NAME" x="47.382" y="17.406" size="1.27" layer="25" rot="R270"/>
+<attribute name="VALUE" x="39.508" y="17.279" size="1.27" layer="27" rot="R270"/>
+</element>
+<element name="D2" library="1_DIOD" package="DIOD" value="SS36C" x="35.62" y="13.44" smashed="yes" rot="R90">
+<attribute name="NAME" x="32.349" y="9.745" size="1.27" layer="25" rot="R90"/>
+<attribute name="VALUE" x="40.109" y="9.954" size="1.27" layer="27" rot="R90"/>
 </element>
 <element name="DD1" library="1_MICRO" package="SOP-8" value="CN3302" x="12.85" y="12.34" smashed="yes" rot="R270">
@@
 <contactref element="VT2" pad="P$7"/>
 <contactref element="VT2" pad="P$8"/>
-<wire x1="25.255" y1="20.62" x2="20.35" y2="22.66" width="0" layer="19" extent="1-1"/>
+<wire x1="20.35" y1="22.66" x2="35.62" y2="16.745" width="0" layer="19" extent="1-1"/>
 <wire x1="18.11" y1="15.195" x2="20.35" y2="22.66" width="0" layer="19" extent="1-1"/>
 <wire x1="18.11" y1="13.925" x2="18.11" y2="15.195" width="0" layer="19" extent="1-1"/>
@@
 <contactref element="VT1" pad="P$4"/>
 <contactref element="VT1" pad="P$9"/>
-<wire x1="30.675" y1="15.75" x2="36.08" y2="16.229" width="0" layer="19" extent="1-1"/>
+<wire x1="30.675" y1="15.75" x2="44.08" y2="17.229" width="0" layer="19" extent="1-1"/>
 <wire x1="29.405" y1="15.75" x2="30.675" y2="15.75" width="0" layer="19" extent="1-1"/>
 <wire x1="28.135" y1="15.75" x2="29.405" y2="15.75" width="0" layer="19" extent="1-1"/>
@@
 <contactref element="C3" pad="P$2"/>
 <contactref element="C4" pad="P$2"/>
-<wire x1="37.929" y1="20.1" x2="38.049" y2="22.55" width="0" layer="19" extent="1-1"/>
-<wire x1="33.879" y1="22.61" x2="38.049" y2="22.55" width="0" layer="19" extent="1-1"/>
-<wire x1="33.909" y1="20.27" x2="33.879" y2="22.61" width="0" layer="19" extent="1-1"/>
-<wire x1="31.865" y1="20.62" x2="33.909" y2="20.27" width="0" layer="19" extent="1-1"/>
-<wire x1="29.405" y1="10.45" x2="31.865" y2="20.62" width="0" layer="19" extent="1-1"/>
+<wire x1="38.661" y1="20.45" x2="43.121" y2="20.39" width="0" layer="19" extent="1-1"/>
+<wire x1="34.821" y1="20.33" x2="38.661" y2="20.45" width="0" layer="19" extent="1-1"/>
+<wire x1="30.581" y1="20.2" x2="34.821" y2="20.33" width="0" layer="19" extent="1-1"/>
+<wire x1="29.405" y1="10.45" x2="30.581" y2="20.2" width="0" layer="19" extent="1-1"/>
 <wire x1="28.08" y1="10.45" x2="29.405" y2="10.45" width="0" layer="19" extent="1-1"/>
 <wire x1="26.851" y1="10.45" x2="28.08" y2="10.45" width="0" layer="19" extent="1-1"/>
+<wire x1="35.62" y1="10.135" x2="29.405" y2="10.45" width="0" layer="19" extent="1-1"/>
 <wire x1="10.45" y1="10.435" x2="26.851" y2="10.45" width="0" layer="19" extent="1-1"/>
 <wire x1="7.7" y1="10.408" x2="10.45" y2="10.435" width="0" layer="19" extent="1-1"/>
@@
 <contactref element="DD1" pad="5"/>
 <contactref element="R6" pad="P$2"/>
-<wire x1="23.352" y1="9.47" x2="15.25" y2="10.435" width="0" layer="19" extent="1-1"/>
+<wire x1="15.25" y1="10.435" x2="23.352" y2="9.47" width="0" layer="19" extent="1-1"/>
 </signal>
 <signal name="N$9">
@@
 <contactref element="C7" pad="P$1"/>
 <contactref element="C6" pad="P$1"/>
-<wire x1="40.404" y1="20.1" x2="40.524" y2="22.55" width="0" layer="19" extent="1-1"/>
-<wire x1="36.354" y1="22.61" x2="40.524" y2="22.55" width="0" layer="19" extent="1-1"/>
-<wire x1="36.384" y1="20.27" x2="36.354" y2="22.61" width="0" layer="19" extent="1-1"/>
-<wire x1="36.08" y1="9.495" x2="36.384" y2="20.27" width="0" layer="19" extent="1-1"/>
-<wire x1="10.45" y1="11.705" x2="36.08" y2="9.495" width="0" layer="19" extent="1-1"/>
+<wire x1="36.186" y1="20.45" x2="40.646" y2="20.39" width="0" layer="19" extent="1-1"/>
+<wire x1="32.346" y1="20.33" x2="36.186" y2="20.45" width="0" layer="19" extent="1-1"/>
+<wire x1="28.106" y1="20.2" x2="32.346" y2="20.33" width="0" layer="19" extent="1-1"/>
+<wire x1="44.08" y1="10.495" x2="40.646" y2="20.39" width="0" layer="19" extent="1-1"/>
+<wire x1="10.45" y1="11.705" x2="28.106" y2="20.2" width="0" layer="19" extent="1-1"/>
 </signal>
 <signal name="N$4">
@@
 <wire x1="23.31" y1="13.925" x2="23.31" y2="15.195" width="0" layer="19" extent="1-1"/>
 <wire x1="23.31" y1="12.655" x2="23.31" y2="13.925" width="0" layer="19" extent="1-1"/>
-<wire x1="15.25" y1="14.245" x2="23.31" y2="12.655" width="0" layer="19" extent="1-1"/>
+<wire x1="15.25" y1="14.245" x2="23.31" y2="13.925" width="0" layer="19" extent="1-1"/>
 <wire x1="14.29" y1="20.44" x2="15.25" y2="14.245" width="0" layer="19" extent="1-1"/>
 </signal>
