File: shema.brd (EAGLE design)
At the start: 100 x 80 mm, 20 parts

Commit message: изменения файлов
Parts:
- moved C4 27.6 mm to (10.0, 7.22)
- moved C3 25.0 mm to (10.0, 10.1), turned to 0 degrees
- moved C2 24.0 mm to (10.0, 13.1)
- moved R6 23.5 mm to (27.4, 5.28), turned to 180 degrees
- moved VT2 22.2 mm to (29.7, 11.2)
- moved VT1 22.0 mm to (38.2, 8.22), turned to 270 degrees
- moved C1 21.1 mm to (9.98, 16.1)
- moved DD1 19.7 mm to (21.9, 7.19), turned to 270 degrees
- moved C5 19.3 mm to (44.8, 6.72)
- moved R4 17.0 mm to (14.3, 14.1)
- moved D1 16.4 mm to (39.9, 17.5), turned to 90 degrees
- moved C6 16.0 mm to (47.7, 6.66)
- moved LED1 15.9 mm to (14.4, 11.4), turned to 0 degrees
- moved L1 15.8 mm to (31.0, 18.1)
- moved RCS 15.3 mm to (11.5, 20.3)
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Routing:
- net GND: track 0.00 -> 109.3 mm, vias 0 -> 8
- net 8.4V: track 0.00 -> 70.6 mm, vias 0 -> 3
- net V_IN: track 0.00 -> 54.1 mm, vias 0 -> 3
- net N$4: track 0.00 -> 29.7 mm, vias 0 -> 2
- net N$6: track 0.00 -> 27.1 mm
- net N$5: track 0.00 -> 20.2 mm
- net N$9: track 0.00 -> 7.99 mm
- net N$11: track 0.00 -> 7.29 mm
- net N$1: track 0.00 -> 5.79 mm
- net N$10: track 0.00 -> 5.41 mm
- net N$12: track 0.00 -> 3.05 mm
- net N$8: track 0.00 -> 2.38 mm
Other:
- board size 100 x 80 mm -> 55 x 25 mm

Commit message: новые файлы
Parts:
- moved R5 0.58 mm to (14.5, 9.38)
- moved D1 0.28 mm to (40.0, 17.7)
Routing:
- net N$6: track 27.1 -> 28.4 mm

Commit message: новые файлы
Parts:
- moved L1 2.02 mm to (29.0, 18.0)
- moved C0 1.00 mm to (44.1, 11.0)
- moved D1 0.99 mm to (39.0, 17.9)
- moved C7 0.90 mm to (47.0, 11.0)
- moved C5 0.71 mm to (44.1, 6.75)
- moved C6 0.58 mm to (47.1, 6.72)
Routing:
- net 8.4V: track 70.3 -> 68.0 mm
- net N$5: track 20.2 -> 18.6 mm
- net GND: track 109.3 -> 108.2 mm
- net N$6: track 28.4 -> 29.5 mm
Other:
- board size 55 x 25 mm -> 53.6 x 25 mm

Commit message: изменения файлов
Parts:
- moved D1 1.31 mm to (38.0, 17.1)
Routing:
- net N$6: track 29.5 -> 27.2 mm
Changed lines of the file:
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@@
 <attribute name="VALUE" x="45.72" y="12.56" size="0.4064" layer="27" rot="R270"/>
 </element>
-<element name="D1" library="1_DIOD" package="CB417-15" value="B560C-13-F" x="39.041" y="17.935" smashed="yes" rot="R90">
-<attribute name="NAME" x="35.87" y="21.767" size="0.4" layer="25"/>
-<attribute name="VALUE" x="43.613" y="14.506" size="1.27" layer="27" rot="R90"/>
+<element name="D1" library="1_DIOD" package="CB417-15" value="B560C-13-F" x="38.029" y="17.109" smashed="yes" rot="R90">
+<attribute name="NAME" x="34.858" y="20.941" size="0.4" layer="25"/>
+<attribute name="VALUE" x="42.601" y="13.68" size="1.27" layer="27" rot="R90"/>
 </element>
 <element name="D2" library="1_DIOD" package="DIOD" value="SS36C" x="21.33" y="17.53" smashed="yes" rot="R270">
@@
 <wire x1="24.3" y1="7.825" x2="19.5" y2="7.825" width="0.45" layer="1"/>
 <wire x1="19.5" y1="7.825" x2="17.9326" y2="7.825" width="0.45" layer="1"/>
-<wire x1="17.7076" y1="8.05" x2="17.9326" y2="7.825" width="0.6096" layer="1"/>
-<via x="17.7076" y="8.05" extent="1-16" drill="0.6" diameter="0.44"/>
+<wire x1="17.7076" y1="8.05" x2="17.9326" y2="7.825" width="0.45" layer="1"/>
+<via x="17.7076" y="8.05" extent="1-16" drill="0.35"/>
 <wire x1="17.7076" y1="8.05" x2="16.7076" y2="7.05" width="0.45" layer="16"/>
-<via x="6.81" y="7.168" extent="1-16" drill="0.6" diameter="0.55"/>
+<via x="6.81" y="7.168" extent="1-16" drill="0.35"/>
 <wire x1="13.3112625" y1="18.08" x2="6.736" y2="18.08" width="0.6096" layer="1"/>
 <wire x1="8.746" y1="16.07" x2="6.736" y2="16.07" width="0.6" layer="1"/>
@@
 <contactref element="VT1" pad="P$4"/>
 <contactref element="VT1" pad="P$9"/>
-<wire x1="39.6235" y1="14.05" x2="38.6755625" y2="14.05" width="0.6096" layer="1"/>
-<wire x1="38.6755625" y1="14.05" x2="38.535" y2="14.05" width="0.6096" layer="1"/>
-<wire x1="38.7305125" y1="12.1538125" x2="34.22" y2="12.160478125" width="0.6" layer="1"/>
-<wire x1="34.22" y1="12.160478125" x2="34.22" y2="18.038" width="0.6" layer="1"/>
+<wire x1="33.845" y1="12.16103125" x2="38.000228125" y2="12.154890625" width="0.6" layer="1"/>
+<wire x1="33.845" y1="12.16103125" x2="33.845" y2="18.038" width="0.6" layer="1"/>
 <wire x1="40.86" y1="6.315" x2="40.86" y2="7.585" width="0.6096" layer="1"/>
 <wire x1="40.86" y1="7.585" x2="40.86" y2="8.855" width="0.6096" layer="1"/>
 <wire x1="38.845" y1="8.22" x2="40.75" y2="10.125" width="0.6096" layer="1"/>
 <wire x1="40.75" y1="10.125" x2="40.86" y2="10.125" width="0.6096" layer="1"/>
-<wire x1="39.6235" y1="14.05" x2="39.6235" y2="12.9015" width="0.6096" layer="1"/>
 <wire x1="40.86" y1="10.125" x2="40.86" y2="11.665" width="0.6096" layer="1"/>
-<wire x1="40.86" y1="11.665" x2="39.6235" y2="12.9015" width="0.6096" layer="1"/>
-<wire x1="34.22" y1="18.038" x2="31.782" y2="18.038" width="0.6" layer="1"/>
-<wire x1="38.6755625" y1="14.05" x2="38.7305125" y2="12.1538125" width="0.6096" layer="1"/>
-<wire x1="39.041" y1="14.556" x2="38.535" y2="14.05" width="0.6096" layer="1"/>
+<wire x1="33.845" y1="18.038" x2="31.782" y2="18.038" width="0.6" layer="1"/>
 <wire x1="40.225" y1="8.22" x2="40.86" y2="8.855" width="0.6" layer="1"/>
 <wire x1="38.845" y1="8.22" x2="40.225" y2="8.22" width="0.6" layer="1"/>
 <wire x1="40.225" y1="8.22" x2="40.86" y2="7.585" width="0.6" layer="1"/>
+<wire x1="40.86" y1="11.665" x2="40.3711875" y2="12.1538125" width="0.6" layer="1"/>
+<wire x1="40.3711875" y1="12.1538125" x2="39" y2="12.1538125" width="0.6" layer="1"/>
+<wire x1="39" y1="12.1538125" x2="38.029" y2="13.1248125" width="0.6" layer="1"/>
+<wire x1="38.029" y1="13.1248125" x2="38.029" y2="13.73" width="0.6" layer="1"/>
+<wire x1="38.000228125" y1="12.154890625" x2="38.00130625" y2="12.1538125" width="0.6" layer="1"/>
+<wire x1="38.00130625" y1="12.1538125" x2="39" y2="12.1538125" width="0.6" layer="1"/>
 </signal>
 <signal name="GND">
@@
 <wire x1="11.82" y1="7.24" x2="11.251" y2="7.24" width="0.8128" layer="1"/>
 <wire x1="19.5" y1="5.285" x2="14.882" y2="5.285" width="0.6096" layer="1"/>
-<via x="31.685" y="6.4564" extent="1-16" drill="0.7" diameter="0.55"/>
+<via x="31.685" y="6.4564" extent="1-16" drill="0.35"/>
 <wire x1="31.685" y1="6.4564" x2="29.2786" y2="4.05" width="0.6096" layer="16"/>
 <wire x1="29.2786" y1="4.05" x2="21.22" y2="4.05" width="0.6096" layer="16"/>
-<via x="21.22" y="4.05" extent="1-16" drill="0.7" diameter="0.55"/>
+<via x="21.22" y="4.05" extent="1-16" drill="0.35"/>
 <wire x1="21.22" y1="4.05" x2="19.5" y2="4.05" width="0.6096" layer="1"/>
 <wire x1="19.5" y1="4.05" x2="19.5" y2="5.285" width="0.6096" layer="1"/>
@@
 <wire x1="44.095" y1="5.511" x2="41.119" y2="2.535" width="0.6" layer="1"/>
 <wire x1="41.119" y1="2.535" x2="35.21" y2="2.535" width="0.6" layer="1"/>
-<via x="35.21" y="2.535" extent="1-16" drill="0.7" diameter="0.55"/>
+<via x="35.21" y="2.535" extent="1-16" drill="0.35"/>
 <wire x1="33.13" y1="4.615" x2="33.13" y2="8.955" width="0.6" layer="16"/>
 <wire x1="35.21" y1="2.535" x2="33.13" y2="4.615" width="0.6096" layer="16"/>
@@
 <wire x1="13.35" y1="6.817" x2="12.927" y2="7.24" width="0.6096" layer="1"/>
 <wire x1="12.927" y1="7.24" x2="11.82" y2="7.24" width="0.6" layer="1"/>
-<via x="17.22" y="16.05" extent="1-16" drill="0.7" diameter="0.55"/>
+<via x="17.22" y="16.05" extent="1-16" drill="0.35"/>
 <wire x1="17.22" y1="16.05" x2="12.75" y2="16.05" width="0.6096" layer="16"/>
 <wire x1="12.75" y1="16.05" x2="12.685" y2="15.985" width="0.6096" layer="16"/>
 <wire x1="12.685" y1="15.985" x2="12.58" y2="16.09" width="0.6096" layer="16"/>
-<via x="12.58" y="16.09" extent="1-16" drill="0.7" diameter="0.55"/>
+<via x="12.58" y="16.09" extent="1-16" drill="0.35"/>
 <wire x1="11.221" y1="16.07" x2="11.241" y2="16.09" width="0.6096" layer="1"/>
 <wire x1="12.58" y1="16.09" x2="11.241" y2="16.09" width="0.6" layer="1"/>
@@
 <wire x1="47.043" y1="12.274" x2="44.165" y2="12.274" width="0.45" layer="1"/>
 <wire x1="44.165" y1="12.274" x2="44.097" y2="12.206" width="0.6096" layer="1"/>
-<wire x1="45.075" y1="13.184" x2="45.075" y2="21.62" width="0.6" layer="1"/>
-<wire x1="44.097" y1="12.206" x2="45.075" y2="13.184" width="0.6" layer="1"/>
-<wire x1="39.041" y1="21.62" x2="39.041" y2="21.29" width="0.6096" layer="1"/>
+<wire x1="44.075" y1="21.62" x2="44.075" y2="12.228" width="0.6" layer="1"/>
+<wire x1="44.097" y1="12.206" x2="44.075" y2="12.228" width="0.6" layer="1"/>
+<wire x1="38.029" y1="21.62" x2="38.029" y2="20.464" width="0.6096" layer="1"/>
 <wire x1="47.133" y1="7.958" x2="44.123" y2="7.958" width="0.45" layer="1"/>
 <wire x1="44.095" y1="7.986" x2="44.123" y2="7.958" width="0.45" layer="1"/>
@@
 <wire x1="19.5" y1="6.555" x2="19.472925" y2="6.582075" width="0.6096" layer="1"/>
 <wire x1="19.472925" y1="6.582075" x2="17.9906" y2="6.582075" width="0.45" layer="1"/>
-<via x="17.9906" y="6.582075" extent="1-16" drill="0.6" diameter="0.55"/>
+<via x="17.9906" y="6.582075" extent="1-16" drill="0.35"/>
 <wire x1="17.9906" y1="6.582075" x2="17.9906" y2="2.7716" width="0.45" layer="16"/>
 <wire x1="18.001" y1="2.7612" x2="18.22" y2="2.5422" width="0.45" layer="16"/>
-<via x="18.22" y="2.5422" extent="1-16" drill="0.6" diameter="0.55"/>
+<via x="18.22" y="2.5422" extent="1-16" drill="0.35"/>
 <wire x1="18.22" y1="2.5422" x2="33.283275" y2="2.5422" width="0.45" layer="1"/>
 <wire x1="33.283275" y1="2.5422" x2="34.350475" y2="3.6094" width="0.45" layer="1"/>
@@
 <wire x1="42.2782" y1="5.47961875" x2="40.40798125" y2="3.6094" width="0.45" layer="1"/>
 <wire x1="17.9906" y1="2.7716" x2="18.001" y2="2.7612" width="0.1524" layer="16"/>
-<wire x1="45.075" y1="21.62" x2="39.041" y2="21.62" width="0.6" layer="1"/>
+<wire x1="44.075" y1="21.62" x2="38.029" y2="21.62" width="0.6" layer="1"/>
 <wire x1="42.309" y1="11.689" x2="42.309" y2="7.808" width="0.45" layer="1"/>
 <wire x1="42.277" y1="7.776" x2="42.277" y2="5.48081875" width="0.45" layer="1"/>
@@
 <wire x1="31.589" y1="8.589" x2="30.319" y2="8.589" width="0.6" layer="1"/>
 <wire x1="30.319" y1="8.589" x2="30.304" y2="8.589" width="0.6" layer="1"/>
-<via x="29.727" y="6.889" extent="1-16" drill="0.7" diameter="0.55"/>
+<via x="29.727" y="6.889" extent="1-16" drill="0.35"/>
 <wire x1="30.304" y1="8.589" x2="29.049" y2="8.589" width="0.6" layer="1"/>
 <wire x1="29.727" y1="6.889" x2="27.613" y2="6.889" width="0.6" layer="16"/>
 <wire x1="27.613" y1="6.889" x2="26.09" y2="8.412" width="0.6" layer="16"/>
-<via x="26.09" y="8.412" extent="1-16" drill="0.7" diameter="0.55"/>
+<via x="26.09" y="8.412" extent="1-16" drill="0.35"/>
 <wire x1="26.09" y1="8.412" x2="26.09" y2="9.191" width="0.6" layer="1"/>
 <wire x1="26.09" y1="9.191" x2="26.071" y2="9.21" width="0.6" layer="1"/>

Commit message: asd
Parts:
- moved RCS 3.13 mm to (14.6, 19.8), turned to 270 degrees
- moved R5 1.99 mm to (16.5, 9.53)
Routing:
- net V_IN: track 54.1 -> 42.1 mm, vias 3 -> 1
- net N$1: track 5.93 -> 2.90 mm
- net N$11: track 6.83 -> 5.52 mm
- net N$4: track 29.7 -> 30.5 mm
- net 8.4V: track 68.5 -> 69.1 mm
- net GND: track 108.2 -> 107.8 mm, vias 8 -> 9
- added copper zone on layer 1, net GND
- added copper zone on layer 1, net N$6

Commit message: изменение файлов
Parts:
- moved RCS 9.98 mm to (21.5, 12.7), turned to 180 degrees
- moved D2 2.53 mm to (19.5, 19.3), turned to 0 degrees
- moved L1 1.28 mm to (28.7, 19.3)
- moved VT1 1.18 mm to (37.2, 7.60)
- moved D1 1.09 mm to (39.1, 17.0), turned to 0 degrees
Routing:
- net GND: track 107.8 -> 131.1 mm, vias 9 -> 13
- net 8.4V: track 69.1 -> 51.2 mm, vias 3 -> 1
- net N$4: track 30.5 -> 14.4 mm
- net N$5: track 18.6 -> 13.2 mm
- net N$6: track 27.2 -> 29.4 mm
- net N$9: track 7.99 -> 6.72 mm
- net V_IN: track 42.1 -> 42.8 mm
- net N$10: track 5.41 -> 4.80 mm
- added copper zone on layer 16, net GND
Other:
- board text added: "GND"
- board text added: "VIN"

Commit message: brd
Routing:
- net V_IN: track 42.8 -> 46.1 mm
- net N$6: track 29.4 -> 28.1 mm, vias 0 -> 14
- net GND: track 131.1 -> 131.3 mm, vias 13 -> 15
Changed lines of the file:
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@@
 <drawing>
 <settings>
-<setting alwaysvectorfont="no"/>
+<setting alwaysvectorfont="yes"/>
 <setting verticaltext="up"/>
 </settings>
@@
 <wire x1="9.36" y1="18.006" x2="8.746" y2="17.392" width="1.27" layer="1"/>
 <wire x1="14.2142625" y1="16.8687375" x2="14.254" y2="16.829" width="1.27" layer="1"/>
-<wire x1="14.254" y1="16.829" x2="14.254" y2="15.256" width="1.27" layer="1"/>
+<wire x1="14.254" y1="15.983" x2="14.254" y2="15.256" width="1.27" layer="1"/>
 <wire x1="14.254" y1="15.256" x2="14.256" y2="15.254" width="0.6096" layer="1"/>
 <wire x1="14.26" y1="14.738" x2="14.256" y2="15.254" width="0.6096" layer="1"/>
@@
 <wire x1="18.668" y1="12.659" x2="22" y2="9.327" width="0.6" layer="1"/>
 <wire x1="22" y1="9.327" x2="22" y2="8.082" width="0.6" layer="1"/>
-<wire x1="17.588" y1="12.649" x2="15.494" y2="14.743" width="0.6" layer="1"/>
+<wire x1="17.588" y1="12.649" x2="16.618" y2="13.619" width="0.6" layer="1"/>
+<wire x1="16.618" y1="13.619" x2="15.494" y2="14.743" width="0.6" layer="1"/>
+<wire x1="14.254" y1="16.829" x2="14.254" y2="15.983" width="1.27" layer="1"/>
+<wire x1="14.254" y1="15.983" x2="16.618" y2="13.619" width="1.27" layer="1"/>
 </signal>
 <signal name="N$5">
@@
 <contactref element="VT1" pad="P$9"/>
 <wire x1="39.852" y1="5.696" x2="39.852" y2="6.966" width="0.6096" layer="1"/>
-<wire x1="39.852" y1="6.966" x2="39.852" y2="8.236" width="0.6096" layer="1"/>
 <wire x1="37.837" y1="7.601" x2="39.742" y2="9.506" width="0.6096" layer="1"/>
 <wire x1="39.742" y1="9.506" x2="39.852" y2="9.506" width="0.6096" layer="1"/>
@@
 <wire x1="32.71" y1="19.29" x2="31.521" y2="19.29" width="0.6096" layer="1"/>
 <wire x1="34.029" y1="16.971" x2="33" y2="18" width="0.6096" layer="1"/>
+<via x="36.181" y="9.032" extent="1-16" drill="0.35"/>
+<via x="36.17" y="8.117" extent="1-16" drill="0.35"/>
+<via x="37.106" y="8.123" extent="1-16" drill="0.35"/>
+<via x="38.037" y="8.123" extent="1-16" drill="0.35"/>
+<via x="38.962" y="8.118" extent="1-16" drill="0.35"/>
+<via x="36.213" y="7.208" extent="1-16" drill="0.35"/>
+<via x="37.139" y="7.208" extent="1-16" drill="0.35"/>
+<via x="38.032" y="7.218" extent="1-16" drill="0.35"/>
+<via x="38.952" y="7.207" extent="1-16" drill="0.35"/>
+<via x="36.234" y="6.304" extent="1-16" drill="0.35"/>
+<via x="37.149" y="6.308" extent="1-16" drill="0.35"/>
+<via x="38.064" y="6.298" extent="1-16" drill="0.35"/>
+<via x="38.979" y="6.298" extent="1-16" drill="0.35"/>
+<via x="37.096" y="9.042" extent="1-16" drill="0.35"/>
 <wire x1="35.521" y1="16.762" x2="35.703584375" y2="16.944584375" width="0" layer="19" extent="1-1"/>
 </signal>
@@
 <wire x1="47.043" y1="9.799" x2="44.165" y2="9.799" width="0.6096" layer="1"/>
 <wire x1="44.165" y1="9.799" x2="44.097" y2="9.731" width="0.6096" layer="1"/>
-<wire x1="50.846" y1="11" x2="49.18" y2="10.2985125" width="0.6" layer="1"/>
-<wire x1="49.18" y1="9.47" x2="49.18" y2="10.2985125" width="0.6" layer="1"/>
+<wire x1="50.846" y1="11" x2="49.725" y2="11" width="0.6" layer="1"/>
+<wire x1="49.725" y1="11" x2="49.18" y2="10.455" width="0.6" layer="1"/>
 <wire x1="49.18" y1="9.47" x2="47.372" y2="9.47" width="0.6" layer="1"/>
 <wire x1="47.372" y1="9.47" x2="47.043" y2="9.799" width="0.6096" layer="1"/>
@@
 <wire x1="34.552" y1="8.291" x2="34.552" y2="6.966" width="0.6096" layer="1"/>
 <wire x1="47.133" y1="5.483" x2="49.18" y2="7.53" width="0.6096" layer="1"/>
-<wire x1="49.18" y1="7.53" x2="49.18" y2="9.47" width="0.6096" layer="1"/>
+<wire x1="49.18" y1="7.53" x2="49.18" y2="10.455" width="0.6096" layer="1"/>
 <wire x1="13.35" y1="6.817" x2="12.927" y2="7.24" width="0.6096" layer="1"/>
 <wire x1="12.927" y1="7.24" x2="12.733" y2="7.24" width="0.6" layer="1"/>
@@
 <wire x1="48.587" y1="14.413" x2="48.587" y2="16.413" width="0.6" layer="16"/>
 <wire x1="50.846" y1="12.154" x2="48.587" y2="14.413" width="0.6" layer="16"/>
-<wire x1="19.5" y1="5.265" x2="19.5" y2="5.285" width="0" layer="19" extent="1-1"/>
-<wire x1="13" y1="5" x2="13.009303125" y2="5.015015625" width="0" layer="19" extent="1-1"/>
+<via x="34" y="22" extent="1-16" drill="0.35"/>
+<via x="22.555" y="6.345" extent="1-16" drill="0.35"/>
 </signal>
 <signal name="N$8">
@@
 <contactref element="VT2" pad="P$4"/>
 <wire x1="27.779" y1="8.589" x2="27.779" y2="7.779" width="0.6" layer="1"/>
-<wire x1="26.555" y1="6.555" x2="24.3" y2="6.555" width="0.6" layer="1"/>
+<wire x1="26.555" y1="6.555" x2="24.3" y2="6.555" width="0.45" layer="1"/>
 <wire x1="27.779" y1="7.779" x2="26.555" y2="6.555" width="0.6" layer="1"/>
 </signal>
@@
 </signal>
 <signal name="N$3">
-<via x="3.022" y="3.029" extent="1-16" drill="3" diameter="6"/>
+<via x="3" y="3" extent="1-16" drill="3" diameter="6"/>
 </signal>
 <signal name="N$16">
@@
 <via x="50.581" y="2.98" extent="1-16" drill="3" diameter="6"/>
 </signal>
-<signal name="N$7">
-<via x="36.181" y="9.032" extent="1-16" drill="0.35"/>
-<via x="36.17" y="8.117" extent="1-16" drill="0.35"/>
-<via x="37.106" y="8.123" extent="1-16" drill="0.35"/>
-<via x="38.037" y="8.123" extent="1-16" drill="0.35"/>
-<via x="38.962" y="8.118" extent="1-16" drill="0.35"/>
-<via x="36.213" y="7.208" extent="1-16" drill="0.35"/>
-<via x="37.139" y="7.208" extent="1-16" drill="0.35"/>
-<via x="38.032" y="7.218" extent="1-16" drill="0.35"/>
-<via x="38.952" y="7.207" extent="1-16" drill="0.35"/>
-<via x="36.234" y="6.304" extent="1-16" drill="0.35"/>
-<via x="37.149" y="6.308" extent="1-16" drill="0.35"/>
-<via x="38.064" y="6.298" extent="1-16" drill="0.35"/>
-<via x="38.979" y="6.298" extent="1-16" drill="0.35"/>
-<wire x1="38.952" y1="7.207" x2="38.962" y2="8.118" width="0" layer="19" extent="1-1"/>
-<wire x1="38.979" y1="6.298" x2="38.952" y2="7.207" width="0" layer="19" extent="1-1"/>
-<wire x1="38.032" y1="7.218" x2="38.952" y2="7.207" width="0" layer="19" extent="1-1"/>
-<wire x1="37.139" y1="7.208" x2="38.032" y2="7.218" width="0" layer="19" extent="1-1"/>
-<wire x1="37.106" y1="8.123" x2="37.139" y2="7.208" width="0" layer="19" extent="1-1"/>
-<wire x1="38.037" y1="8.123" x2="38.032" y2="7.218" width="0" layer="19" extent="1-1"/>
-<wire x1="37.149" y1="6.308" x2="37.139" y2="7.208" width="0" layer="19" extent="1-1"/>
-<wire x1="36.234" y1="6.304" x2="37.149" y2="6.308" width="0" layer="19" extent="1-1"/>
-<wire x1="36.213" y1="7.208" x2="36.234" y2="6.304" width="0" layer="19" extent="1-1"/>
-<wire x1="36.17" y1="8.117" x2="36.213" y2="7.208" width="0" layer="19" extent="1-1"/>
-<wire x1="36.181" y1="9.032" x2="36.17" y2="8.117" width="0" layer="19" extent="1-1"/>
-<wire x1="38.064" y1="6.298" x2="38.979" y2="6.298" width="0" layer="19" extent="1-1"/>
-</signal>
-<signal name="N$13">
-<via x="37.096" y="9.042" extent="1-16" drill="0.35"/>
-</signal>
 <signal name="N$14">

Commit message: изменение файлов
Parts:
- moved C7 6.21 mm to (45.8, 17.1), turned to 180 degrees
- moved C6 5.91 mm to (46.0, 12.5), turned to 180 degrees
- moved C0 4.23 mm to (45.9, 14.8), turned to 180 degrees
- moved C5 3.80 mm to (46.0, 10.0), turned to 180 degrees
- moved D1 2.24 mm to (38.1, 19.0)
Routing:
- net GND: track 131.3 -> 143.8 mm, vias 15 -> 16
- net V_IN: track 46.1 -> 48.0 mm
- net N$6: track 28.1 -> 29.0 mm, vias 14 -> 16
- net 8.4V: track 51.2 -> 50.6 mm
Other:
- board size 53.6 x 25 mm -> 55 x 25.1 mm
